File: EDA/EDA.kicad_sch (KiCad schematic)
At the start: 39 parts, among them J1 USB_B, J2 Conn_01x20_Pin, SW1 SW_Push, U1 ATmega328PB-A, U2 CP2102N-Axx-xQFN24, U3 NCP1117-3.3_SOT223, U4 DRV8837, U5 DRV8837, U6 BMI160, Y2 Crystal_GND24

Commit message: New USB design, w/ cheched
Parts:
- removed Y2: Crystal_GND24, Crystal:Crystal_SMD_3225-4Pin_3.2x2.5mm, symbol Device:Crystal_GND24
- added C10, C11: 22pF, Capacitor_SMD:C_0805_2012Metric_Pad1.18x1.45mm_HandSolder, symbol Device:C
- added C12, C14, C16: 100nF, Capacitor_SMD:C_0805_2012Metric_Pad1.18x1.45mm_HandSolder, symbol Device:C
- added C13, C15: 4.7uF, Capacitor_SMD:C_0805_2012Metric_Pad1.18x1.45mm_HandSolder, symbol Device:C
- added D6: D_Zener, Diode_SMD:D_0603_1608Metric_Pad1.05x0.95mm_HandSolder, symbol Device:D_Zener
- added D8: SP0503BAHT, Package_TO_SOT_SMD:SOT-143_Handsoldering, symbol Power_Protection:SP0503BAHT
- added J3: USB_B, Connector_USB:USB_B_OST_USB-B1HSxx_Horizontal, symbol Connector:USB_B
- added R13: 4.7k, Resistor_SMD:R_0603_1608Metric_Pad0.98x0.95mm_HandSolder, symbol Device:R
- added R14: 22.1k, Resistor_SMD:R_0603_1608Metric_Pad0.98x0.95mm_HandSolder, symbol Device:R
- added R15: 47.5k, Resistor_SMD:R_0603_1608Metric_Pad0.98x0.95mm_HandSolder, symbol Device:R
- added R16, R17, R18, R19, R20: 1k, Resistor_SMD:R_0603_1608Metric_Pad0.98x0.95mm_HandSolder, symbol Device:R
- added RX, TX: LED, LED_SMD:LED_0603_1608Metric_Pad1.05x0.95mm_HandSolder, symbol Device:LED
- added SW2: SW_Push, symbol Switch:SW_Push
- added U7: ATmega328PB-A, Package_QFP:TQFP-32_7x7mm_P0.8mm, symbol MCU_Microchip_ATmega:ATmega328PB-A
- added U8: CP2102N-Axx-xQFN24, Package_DFN_QFN:QFN-24-1EP_4x4mm_P0.5mm_EP2.6x2.6mm, symbol Interface_USB:CP2102N-Axx-xQFN24
- added Y1: Crystal, Crystal:Crystal_SMD_HC49-SD_HandSoldering, symbol Device:Crystal
Connections:
- net DTR: now also U8.23 (~{DTR})
- net GND: now also C10.2, C11.2, C12.2, C13.2, C14.2, C15.2, C16.2, D8.1 (A), J3.4 (GND), J3.5 (Shield), R15.2, SW2.2, U7.21 (GND), U7.5 (GND), U8.2 (GND), U8.25 (GND)
- net RXD: now also R18.2
- net TXD: now also R17.2
- net VCC: now also D6.1 (K), R13.1, U7.18 (AVCC), U7.4 (VCC)
- new net: TX.1 (K), U8.13 (~{RXT}/GPIO.1)
- new net: RX.1 (K), U8.14 (~{TXT}/GPIO.0)
- new net: R18.1, U8.20 (RXD)
- new net: R17.1, U8.21 (TXD)
- new net: D8.2 (K), J3.2 (D-), U8.3 (D+)
- new net: D8.3 (K), J3.3 (D+), U8.4 (D-)
- new net: C15.1, C16.1, R16.2, R19.1, R20.1, U8.5 (VIO), U8.6 (VDD)
- new net: C13.1, C14.1, D8.4 (K), J3.1 (VBUS), R14.1, U8.7 (VREGIN)
- new net: R14.2, R15.1, U8.8 (VBUS)
- new net: R16.1, U8.9 (~{RST})
- new net: R20.2, TX.2 (A)
- new net: R19.2, RX.2 (A)
- new net: C11.1, U7.8 (XTAL2/PB7), Y1.1
- new net: C10.1, U7.7 (XTAL1/PB6), Y1.2
- new net: C12.1, D6.2 (A), R13.2, SW2.1, U7.29 (~{RESET}/PC6)
- no-connect marks 18 -> 27
